File: hardware/aurora-ctrl/aurora-ctrl/aurora-ctrl.kicad_sch (KiCad schematic)
At the start: 0 parts

Commit message: M2: TPS5430 12V->5V buck stage wired and annotated, ERC clean
Other:
- added sheet Analog_FE (Analog_FE.kicad_sch)
- added sheet CAN (CAN.kicad_sch)
- added sheet MCU (MCU.kicad_sch)
- added sheet Motor (Motor.kicad_sch)
- added sheet Safety (Safety.kicad_sch)
- added sheet power (power.kicad_sch)
